File: pss.kicad_pcb (KiCad board)
At the start: 2 copper layers, 659 parts, among them J101 Conn_01x06_Socket, J102 Conn_01x02_Socket, J103 Conn_01x02_Socket, J104 Conn_01x02_Socket, J2001 Conn_01x06_Socket, J2002 Conn_01x06_Socket, J2101 Conn_01x06_Socket, J2801 Conn_01x06_Socket, K3501 ALFG2PF12, M2101 Fan, M2801 Fan, Q1401 DNLS350E, Q1901 DPLS350E, Q1902 DNLS350E, Q1903 DPLS350E, Q1904 DPLS350E, Q1905 DNLS350E, Q1906 DNLS350E, Q1907 TIP41C, Q1908 TIP42C, Q2201 DNLS350E, Q2202 DPLS350E, Q2203 TIP41C, Q2204 TIP42C, Q2301 DNLS350E, Q2302 DPLS350E, Q2303 TIP41C, Q2304 TIP42C, Q2401 DNLS350E, Q2402 DPLS350E, Q2403 TIP41C, Q2404 TIP42C, Q2501 DNLS350E, Q2502 DPLS350E, Q2503 TIP41C, Q2504 TIP42C, Q2601 DNLS350E, Q2602 DPLS350E, Q2603 TIP41C, Q2604 TIP42C, Q2701 DNLS350E, Q2702 DPLS350E, Q2703 TIP41C, Q2704 TIP42C, Q2901 DNLS350E, Q2902 DPLS350E, Q2903 TIP41C, Q2904 TIP42C, Q3001 DNLS350E, Q3002 DPLS350E, Q3003 TIP41C, Q3004 TIP42C, Q3101 DNLS350E, Q3102 DPLS350E, Q3103 TIP41C, Q3104 TIP42C, Q3201 DNLS350E, Q3202 DPLS350E, Q3203 TIP41C, Q3204 TIP42C, Q3301 DNLS350E, Q3302 DPLS350E, Q3303 TIP41C, Q3304 TIP42C, Q3401 DNLS350E, Q3402 DPLS350E, Q3403 TIP41C, Q3404 TIP42C, Q3501 DPLS350E, Q401 DNLS350E, Q402 DNLS350E, Q403 DPLS350E, Q404 DPLS350E, U1001 TLV9352, U1101 TLV9352, U1201 TLV9352, U1301 TLV9352, U1401 4081, U1402 4073, U1403 4073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

Commit message: edit pcb soldermask expansion
Other:
- rule pad_to_mask_clearance: 0 -> 0.0762
Changed lines of the file:
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@@
 	)
 	(layers
-		(0 "F.Cu" signal)
-		(31 "B.Cu" signal)
+		(0 "F.Cu" mixed)
+		(31 "B.Cu" mixed)
 		(32 "B.Adhes" user "B.Adhesive")
 		(33 "F.Adhes" user "F.Adhesive")
@@
 		(48 "B.Fab" user)
 		(49 "F.Fab" user)
-		(50 "User.1" user)
-		(51 "User.2" user)
-		(52 "User.3" user)
-		(53 "User.4" user)
-		(54 "User.5" user)
-		(55 "User.6" user)
-		(56 "User.7" user)
-		(57 "User.8" user)
-		(58 "User.9" user)
 	)
 	(setup
-		(pad_to_mask_clearance 0)
+		(stackup
+			(layer "F.SilkS"
+				(type "Top Silk Screen")
+				(color "White")
+				(material "Direct Printing")
+			)
+			(layer "F.Paste"
+				(type "Top Solder Paste")
+			)
+			(layer "F.Mask"
+				(type "Top Solder Mask")
+				(color "Green")
+				(thickness 0.01)
+				(material "Epoxy")
+				(epsilon_r 3.3)
+				(loss_tangent 0)
+			)
+			(layer "F.Cu"
+				(type "copper")
+				(thickness 0.035)
+			)
+			(layer "dielectric 1"
+				(type "core")
+				(color "FR4 natural")
+				(thickness 1.51)
+				(material "FR4")
+				(epsilon_r 4.5)
+				(loss_tangent 0.02)
+			)
+			(layer "B.Cu"
+				(type "copper")
+				(thickness 0.035)
+			)
+			(layer "B.Mask"
+				(type "Bottom Solder Mask")
+				(color "Green")
+				(thickness 0.01)
+				(material "Epoxy")
+				(epsilon_r 3.3)
+				(loss_tangent 0)
+			)
+			(layer "B.Paste"
+				(type "Bottom Solder Paste")
+			)
+			(layer "B.SilkS"
+				(type "Bottom Silk Screen")
+				(color "White")
+				(material "Direct Printing")
+			)
+			(copper_finish "HAL lead-free")
+			(dielectric_constraints no)
+		)
+		(pad_to_mask_clearance 0.0762)
+		(solder_mask_min_width 0.1016)
 		(allow_soldermask_bridges_in_footprints no)
 		(pcbplotparams
@@
 			(size 7 4)
 			(drill oval 5 2)
-			(layers "F&B.Cu" "*.Mask")
+			(layers "*.Cu" "*.Mask")
 		)
 		(pad "" np_thru_hole oval
@@
 			(size 7 4)
 			(drill oval 5 2)
-			(layers "F&B.Cu" "*.Mask")
+			(layers "*.Cu" "*.Mask")
 		)
 		(pad "" np_thru_hole oval
@@
 			(size 7 4)
 			(drill oval 5 2)
-			(layers "F&B.Cu" "*.Mask")
+			(layers "*.Cu" "*.Mask")
 		)
 		(pad "" np_thru_hole oval
@@
 			(size 7 4)
 			(drill oval 5 2)
-			(layers "F&B.Cu" "*.Mask")
+			(layers "*.Cu" "*.Mask")
 		)
 		(pad "1" thru_hole circle
@@
 			(size 7 4)
 			(drill oval 5 2)
-			(layers "F&B.Cu" "*.Mask")
+			(layers "*.Cu" "*.Mask")
 		)
 		(pad "" np_thru_hole oval
@@
 			(size 7 4)
 			(drill oval 5 2)
-			(layers "F&B.Cu" "*.Mask")
+			(layers "*.Cu" "*.Mask")
 		)
 		(pad "" np_thru_hole oval
@@
 			(size 7 4)
 			(drill oval 5 2)
-			(layers "F&B.Cu" "*.Mask")
+			(layers "*.Cu" "*.Mask")
 		)
 		(pad "" np_thru_hole oval
@@
 			(size 7 4)
 			(drill oval 5 2)
-			(layers "F&B.Cu" "*.Mask")
+			(layers "*.Cu" "*.Mask")
 		)
 		(pad "1" thru_hole circle

Commit message: fix soldermask expansion DRC error for bridging
Other:
- rule pad_to_mask_clearance: 0.0762 -> 0
Changed lines of the file:
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@@
 			(dielectric_constraints no)
 		)
-		(pad_to_mask_clearance 0.0762)
-		(solder_mask_min_width 0.1016)
+		(pad_to_mask_clearance 0)
 		(allow_soldermask_bridges_in_footprints no)
 		(pcbplotparams

Commit message: add pcb edge cuts outline and NPTH mounting hole for plug-in unit mounting
Parts:
- added REF**: MountingHole_2.8mm, pss:MountingHole_2.8mm, F.Cu at (305.6, 236.4)
- added REF**: MountingHole_2.8mm, pss:MountingHole_2.8mm, F.Cu at (142.4, 236.4)
- added REF**: MountingHole_2.8mm, pss:MountingHole_2.8mm, F.Cu at (394.4, 236.4)
- added REF**: MountingHole_2.8mm, pss:MountingHole_2.8mm, F.Cu at (279.4, 236.4)
- added REF**: MountingHole_2.8mm, pss:MountingHole_2.8mm, F.Cu at (53.5, 236.4)
- added REF**: MountingHole_2.8mm, pss:MountingHole_2.8mm, F.Cu at (190.6, 236.4)
- moved C1001 321.3 mm to (305.9, -111.7)
- moved C1101 321.3 mm to (235.3, -74.0)
- moved C1201 321.3 mm to (273.1, -111.7)
- moved C1301 321.3 mm to (289.5, -111.7)
- moved C1401 321.3 mm to (192.4, -248.2)
- moved C1402 321.3 mm to (192.4, -245.2)
- moved C1403 321.3 mm to (192.4, -242.2)
- moved C1404 321.3 mm to (192.4, -239.2)
- moved C1405 321.3 mm to (192.4, -236.2)
- moved C1406 321.3 mm to (192.4, -233.2)
- moved C1407 321.3 mm to (192.4, -230.2)
- moved C1408 321.3 mm to (192.4, -227.2)
- moved C1501 321.3 mm to (169.4, -41.8)
- moved C1502 321.3 mm to (169.4, -38.8)
- moved C1503 321.3 mm to (169.4, -35.8)
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Other:
- board outline added: 352 x 220 mm
