File: control-var.kicad_sch (KiCad schematic)
At the start: 58 parts, among them U501 OPA2810, U502 OPA2810, U503 OPA2810

Commit message: edit trimmer adjustment style to sideways
Parts:
- RV501, RV502: footprint pss:Potentiometer_Bourns_PVG5A -> pss:Potentiometer_Bourns_PVG5H; MPN PVG5A103C03B00 -> PVG5H103C03R00; VPN 81-PVG5A103C03B00 -> 81-PVG5H103C03R00
- RV503: footprint pss:Potentiometer_Bourns_PVG5A -> pss:Potentiometer_Bourns_PVG5H; MPN PVG5A104C03B00 -> PVG5H104C03R00; VPN 81-PVG5A104C03B00 -> 81-PVG5H104C03R00
Changed lines of the file:
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@@
 		(title "Power Supply Sink")
 		(date "2024-12-07")
-		(rev "0.13.3")
+		(rev "0.13.4")
 		(company "Open Battery Tester")
 		(comment 1 "Control with variable parameters")
@@
 			)
 		)
-		(property "Footprint" "pss:Potentiometer_Bourns_PVG5A"
+		(property "Footprint" "pss:Potentiometer_Bourns_PVG5H"
 			(at 213.36 124.46 0)
 			(effects
@@
 			)
 		)
-		(property "MPN" "PVG5A104C03B00"
+		(property "MPN" "PVG5H104C03R00"
 			(at 213.36 124.46 0)
 			(effects
@@
 			)
 		)
-		(property "VPN" "81-PVG5A104C03B00"
+		(property "VPN" "81-PVG5H104C03R00"
 			(at 213.36 124.46 0)
 			(effects
@@
 			)
 		)
-		(property "Footprint" "pss:Potentiometer_Bourns_PVG5A"
+		(property "Footprint" "pss:Potentiometer_Bourns_PVG5H"
 			(at 158.75 111.76 0)
 			(effects
@@
 			)
 		)
-		(property "MPN" "PVG5A103C03B00"
+		(property "MPN" "PVG5H103C03R00"
 			(at 158.75 111.76 0)
 			(effects
@@
 			)
 		)
-		(property "VPN" "81-PVG5A103C03B00"
+		(property "VPN" "81-PVG5H103C03R00"
 			(at 158.75 111.76 0)
 			(effects
@@
 			)
 		)
-		(property "Footprint" "pss:Potentiometer_Bourns_PVG5A"
+		(property "Footprint" "pss:Potentiometer_Bourns_PVG5H"
 			(at 191.77 41.91 0)
 			(effects
@@
 			)
 		)
-		(property "MPN" "PVG5A103C03B00"
+		(property "MPN" "PVG5H103C03R00"
 			(at 191.77 41.91 0)
 			(effects
@@
 			)
 		)
-		(property "VPN" "81-PVG5A103C03B00"
+		(property "VPN" "81-PVG5H103C03R00"
 			(at 191.77 41.91 0)
 			(effects
