File: window-comparator.kicad_sch (KiCad schematic)
At the start: 12 parts, among them U1001 TLV9352

Commit message: edit trimmer adjustment style to sideways
Parts:
- RV1001, RV1002: footprint pss:Potentiometer_Bourns_PVG5A -> pss:Potentiometer_Bourns_PVG5H; MPN PVG5A102C03B00 -> PVG5H102C03R00; VPN 81-PVG5A102C03B00 -> 81-PVG5H102C03R00
Changed lines of the file:
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@@
 		(title "Power Supply Sink")
 		(date "2024-12-07")
-		(rev "0.13.3")
+		(rev "0.13.4")
 		(company "Open Battery Tester")
 		(comment 1 "Window-Comparator")
@@
 			)
 		)
-		(property "Footprint" "pss:Potentiometer_Bourns_PVG5A"
+		(property "Footprint" "pss:Potentiometer_Bourns_PVG5H"
 			(at 116.84 109.22 0)
 			(effects
@@
 			)
 		)
-		(property "MPN" "PVG5A102C03B00"
+		(property "MPN" "PVG5H102C03R00"
 			(at 116.84 109.22 0)
 			(effects
@@
 			)
 		)
-		(property "VPN" "81-PVG5A102C03B00"
+		(property "VPN" "81-PVG5H102C03R00"
 			(at 116.84 109.22 0)
 			(effects
@@
 			)
 		)
-		(property "Footprint" "pss:Potentiometer_Bourns_PVG5A"
+		(property "Footprint" "pss:Potentiometer_Bourns_PVG5H"
 			(at 116.84 85.09 0)
 			(effects
@@
 			)
 		)
-		(property "MPN" "PVG5A102C03B00"
+		(property "MPN" "PVG5H102C03R00"
 			(at 116.84 85.09 0)
 			(effects
@@
 			)
 		)
-		(property "VPN" "81-PVG5A102C03B00"
+		(property "VPN" "81-PVG5H102C03R00"
 			(at 116.84 85.09 0)
 			(effects
